File: Undroid.kicad_pcb (KiCad board)
At the start: 6 copper layers, 61.7 x 133.2 mm, 38 parts

Commit message: pcb-master: Fix PCB (MHR-0002)
Signed-off-by: Amlal El Mahrouss <amlal.elmahrouss@icloud.com>
Parts:
- moved JACK_PORT1 2.51 mm to (179.0, 155.5), turned to 0 degrees
Routing:
- net Net-(CPU_1A-GND): track 18.3 -> 0.00 mm
- net SND_IN: track 75.8 -> 91.1 mm
- net GSM_PWR_N: track 56.6 -> 55.0 mm
- net GSM_RST_N: track 90.7 -> 89.2 mm
- net Net-(MBCI_0-VDD): track 62.3 -> 63.4 mm
- net GND: track 223.8 -> 224.8 mm
Other:
- board text added: "MHR-0002"
- board text added: "ZETA"
- board text removed: "Undroid"
- board text removed: "ZETA-0001"

Commit message: Generate gerbers file, fix circuits.
Signed-off-by: Amlal EL Mahrouss <amlalelmahrouss@icloud.com>
Routing:
- net RAM_WE_N: track 54.1 -> 53.6 mm

Commit message: PCB: Improve planes.
Signed-off-by: Amlal EL Mahrouss <amlalelmahrouss@icloud.com>
Routing:
- net GND: track 224.8 -> 296.9 mm, vias 20 -> 25
- net Net-(ANT1-A): track 58.6 -> 61.0 mm, vias 0 -> 2
- net VBUS_USBC: track 228.2 -> 229.1 mm
- added copper zone on F.Cu, net 3.3V
- removed copper zone on In1.Cu, net 3.3V
- removed copper zone on F.Cu, net GND

Commit message: Undroid: Fix PCB.
Signed-off-by: Amlal EL Mahrouss <amlalelmahrouss@icloud.com>
Routing:
- net VBUS_USBC: track 229.1 -> 253.8 mm
- net RTS1: track 101.1 -> 110.6 mm
- net A2: track 111.2 -> 117.3 mm
- net A1: track 129.7 -> 134.5 mm
- net RTC_OUT: track 173.2 -> 177.1 mm
- net GSM_IO: track 87.1 -> 90.9 mm
- net Net-(SIM_CHIP1-NETLIGHT): track 63.0 -> 64.7 mm
- net RAM_CK: track 22.2 -> 23.4 mm
- net Net-(SD_SLOT_1-VDD): track 8.95 -> 9.68 mm
- added copper zone on In2.Cu, net GND
- added copper zone on In3.Cu, net GND
- added copper zone on In4.Cu, net GND

Commit message: MHR-0002: Final revision of PCB before getting sent out.
Signed-off-by: Amlal EL Mahrouss <amlalelmahrouss@icloud.com>
Routing:
- net CPU_PWR: track 76.8 -> 95.3 mm
- net SND_IN: track 91.1 -> 80.2 mm
- net GND: track 296.8 -> 288.8 mm, vias 25 -> 24
- net VBUS_USBC: track 253.8 -> 250.5 mm
- net DTR1: track 30.7 -> 32.2 mm
- net Net-(SIM_CHIP1-NETLIGHT): track 64.7 -> 66.1 mm
- net CTS1: track 46.2 -> 47.5 mm
- net SD_DAT2: track 79.7 -> 78.6 mm
- net A11: track 136.2 -> 135.4 mm
- net Net-(SD_SLOT_1-VDD): track 9.68 -> 9.16 mm
Other:
- board text added: ":)"

Commit message: PCB improvements and generated BoM, Gerbers and reports.
Signed-off-by: Amlal EL Mahrouss <amlalelmahrouss@icloud.com>
Routing:
- net VBUS_USBC: track 250.5 -> 260.1 mm
- net CPU_PWR: track 95.3 -> 96.2 mm
- net Net-(BRIDGE_CHIP1-GND-Pad14): track 55.8 -> 55.0 mm
